File: avlsi_test_boards/power_board/power_board.kicad_pcb (KiCad board)
At the start: 4 copper layers, 100 x 100 mm, 113 parts, among them J1 PJ-102AH, J2 PJ-102AH, J3 Conn_02x07_Odd_Even, J4 Conn_02x07_Odd_Even, J5 Conn_02x20_Odd_Even, J6 Conn_02x20_Odd_Even, J7 Conn_02x20_Odd_Even, J8 Conn_02x20_Odd_Even, U1 TLV1117LV18DCYR, U11 SN74LVC16T245DLR, U12 SN74LVC16T245DLR, U13 SN74LVC16T245DLR, U14 SN74LVC16T245DLR, U15 DS04-254-2-04BK-SMT, U17 SN74LVC16T245DLR, U3 TLV1117LV25DCYR, U4 DS04-254-2-04BK-SMT, U5 74HC4051D_653, U6 TLV75709PDBV, U7 TLV75709PDBV, U8 TLV1117LV33DCYR

Commit message: Add initial layout stuff
Parts:
- added J10: Conn_02x07_Odd_Even, Connector_PinHeader_2.54mm:PinHeader_2x07_P2.54mm_Vertical, F.Cu at (264.1, 15.8)
- added J9: Conn_02x07_Odd_Even, Connector_PinHeader_2.54mm:PinHeader_2x07_P2.54mm_Vertical, B.Cu at (343.1, 40.6)
- added U10: ~, avlsi:opal_kelly_XEM7310_header, B.Cu at (149.5, 104.6)
- added U16: SN74LVC16T245DLR, avlsi:DL48, F.Cu at (79.4, 52.2)
- added U9: TLV1117LV33DCYR, avlsi:VREG_TLV1117LV33DCYR, F.Cu at (310.1, 79.0)
- C1, C11, C12, C13, C15, C16, C17, C18, C19, C2, C20, C21, C3, C4, C5, C6, C7, C8: footprint Capacitor_SMD:C_0603_1608Metric -> Capacitor_SMD:C_0805_2012Metric; moved to F.Cu
- C10, C14, C9: footprint Capacitor_SMD:C_0603_1608Metric -> Capacitor_SMD:C_0805_2012Metric
- C22, C23, C24, C25, C26, C27, C28, C29, C30, C31, C32, C33, C34, C35, C36, C37, C38, C39, C40, C41, C42, C43, C44, C47, C48: moved to F.Cu
- R1, R11, R12, R15, R16, R19, R2, R20, R23, R24, R27, R28, R3, R31, R32, R7, R8: footprint Resistor_SMD:R_0201_0603Metric -> Resistor_SMD:R_0805_2012Metric
- U15: value DS04-254-2-04BK-SMT -> SN74LVC16T245DLR; footprint ds:DS04-254-2-04BK-SMT_CUD -> avlsi:DL48
- U2: value ~ -> TLV1117LV25DCYR; footprint avlsi:opal_kelly_XEM7310_header -> avlsi:SOT230P700X180-4N; moved to F.Cu
- U3: value TLV1117LV25DCYR -> TLV1117LV33DCYR; footprint avlsi:SOT230P700X180-4N -> avlsi:VREG_TLV1117LV33DCYR
- U6: value TLV75709PDBV -> TLV1117LV18DCYR; footprint Package_TO_SOT_SMD:SOT-23-5 -> avlsi:SOT230P700X180-4N
- U8: value TLV1117LV33DCYR -> TLV1117LV25DCYR; footprint avlsi:VREG_TLV1117LV33DCYR -> avlsi:SOT230P700X180-4N
- moved R4 257.9 mm to (335.7, 67.8)
- moved R18 201.5 mm to (276.5, 111.3)
- moved J3 199.9 mm to (321.7, 40.6), turned to 0 degrees
- moved U7 199.8 mm to (328.9, 68.7)
- moved C15 199.6 mm to (320.3, 75.1), turned to 0 degrees
- moved J2 199.2 mm to (332.9, 53.0)
- moved U8 195.8 mm to (310.1, 70.9)
- moved R19 191.7 mm to (266.3, 109.2)
- moved R20 191.7 mm to (266.3, 110.9)
- moved C49 190.6 mm to (260.9, 105.3)
- moved C46 189.0 mm to (260.9, 96.3)
- moved R29 188.2 mm to (260.8, 108.3)
- moved R30 188.2 mm to (260.8, 111.3)
- moved U6 187.8 mm to (310.1, 62.9), turned to 0 degrees
- moved R31 178.1 mm to (250.7, 109.2)
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Connections:
- U15 pad 1: DVIN5 -> /level_shifter4/DIR1
- U15 pad 2: DVIN5 -> MC1_16
- U15 pad 3: DVIN5 -> MC1_18
- U15 pad 4: DVIN5 -> DGND
- U15 pad 5: unconnected-(U15-Pad5) -> MC1_20
- U15 pad 6: /digital_power_converters/S0 -> MC1_22
- U15 pad 7: /digital_power_converters/S1 -> VCCD33
- U15 pad 8: /digital_power_converters/S2 -> MC1_24
- U3 pad 2: /VCCD25 -> VCCD33
- U3 pad 4: /VCCD25 -> VCCD33
- U6 pad 1: /AVIN5 -> ADGND
- U6 pad 2: ADGND -> /VCCA18
- U6 pad 4: unconnected-(U6-NC-Pad4) -> /VCCA18
- U8 pad 2: /VCCA33 -> /VCCA25
- U8 pad 4: /VCCA33 -> /VCCA25
Routing:
- net DGND: track 1158.5 -> 0.00 mm, vias 109 -> 0
- net (no net): track 630.5 -> 0.00 mm, vias 1 -> 0
- net V_Level_Shift: track 536.9 -> 0.00 mm, vias 60 -> 0
- net /pin_header/33VDD: track 196.6 -> 0.00 mm
- net /pin_header/VDCIN: track 164.7 -> 0.00 mm
- net /pin_header/3VDD: track 152.5 -> 0.00 mm
- net DVIN5: track 133.2 -> 0.00 mm, vias 8 -> 0
- net /pin_header/VCCO_MC1: track 131.8 -> 0.00 mm
- net /AVIN5: track 98.0 -> 0.00 mm, vias 8 -> 0
- net /pin_header/10VDD: track 96.7 -> 0.00 mm
- net /pin_header/VCCO_MC2: track 87.7 -> 0.00 mm
- net VCCD33: track 75.3 -> 0.00 mm, vias 5 -> 0
- net MC1_41_PIN: track 71.2 -> 0.00 mm, vias 1 -> 0
- net MC1_43_PIN: track 70.2 -> 0.00 mm, vias 1 -> 0
- net MC1_42_PIN: track 69.0 -> 0.00 mm, vias 1 -> 0
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- removed copper zone on B.Cu, net ADGND
- removed copper zone on F.Cu, net ADGND
- removed copper zone on B.Cu, net DGND
- removed copper zone on F.Cu, net DGND
Other:
- board text added: "VACustom"
- board text added: "VCCA09"
- board text added: "VCCA12"
- board text added: "VCCA18"
- board text added: "VCCA25"
- board text added: "VCCA33"
- board text added: "VIN5"
- board text removed: "DGND"
- board text removed: "EMI?"
- board text removed: "Groudning pull up resistors near switches?"
- board text removed: "Grounding with copper pour?"
- board text removed: "Is it possible to place vias on the pads? could save some space and make things neater but may not be good practice"
- board text removed: "LS1"
- board text removed: "LS2"
- board text removed: "LS3"
- board text removed: "LS4"
- board text removed: "LS5"
- board text removed: "LS6"
- board text removed: "LS7"
- board text removed: "Make central trace thicker to input of level shifter?"
- board text removed: "Maybe the unfilled zone on the back is okay bevause its connected to ground through the back?"
- board text removed: "VA09"
- board text removed: "VA12"
- board text removed: "VA18"
- board text removed: "VA27"
- board text removed: "VA33"
- board text removed: "VA50"
- board text removed: "VCUST"
- board text removed: "VD09"
- board text removed: "VD12"
- board text removed: "VD18"
- board text removed: "VD27"
- board text removed: "VD33"
- board text removed: "VD50"
- board text removed: "Where should analog pins be routed?"
- board text removed: "smoothen traces"

Commit message: Add analog power pins
Parts:
- J9: moved to F.Cu
- U13, U14: moved to B.Cu
- moved U1 189.6 mm to (215.5, 107.2)
- moved U2 189.6 mm to (215.5, 115.2)
- moved U3 189.6 mm to (215.5, 123.3)
- moved VR1 189.6 mm to (215.5, 131.3)
- moved VR2 189.6 mm to (215.5, 139.4)
- moved C13 187.6 mm to (133.9, 48.3), turned to 90 degrees
- moved J9 186.5 mm to (157.0, 28.8), turned to 0 degrees
- moved C15 184.7 mm to (137.5, 48.3), turned to 90 degrees
- moved J2 184.0 mm to (149.3, 41.2)
- moved J3 184.0 mm to (138.1, 28.8)
- moved C12 180.1 mm to (141.2, 48.3), turned to 90 degrees
- moved C14 177.3 mm to (144.7, 48.3), turned to 90 degrees
- moved C18 177.2 mm to (148.5, 48.3), turned to 90 degrees
- moved VR3 176.9 mm to (136.2, 54.5), turned to -90 degrees
- moved C20 174.4 mm to (152.0, 48.3), turned to 90 degrees
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Connections:
- J9 pad 1: /VACustom -> ADGND
- J9 pad 10: ADGND -> /VCCA25
- J9 pad 11: /VCCA33 -> ADGND
- J9 pad 12: ADGND -> /VCCA33
- J9 pad 13: /AVIN5 -> ADGND
- J9 pad 14: ADGND -> /AVIN5
- J9 pad 2: ADGND -> /VACustom
- J9 pad 3: /VCCA09 -> ADGND
- J9 pad 4: ADGND -> /VCCA09
- J9 pad 5: /VCCA12 -> ADGND
- J9 pad 6: ADGND -> /VCCA12
- J9 pad 7: /VCCA18 -> ADGND
- J9 pad 8: ADGND -> /VCCA18
- J9 pad 9: /VCCA25 -> ADGND
Routing:
- net /VCCA25: track 0.00 -> 70.2 mm, vias 0 -> 1
- net /VCCA12: track 0.00 -> 60.1 mm
- net /VCCA18: track 0.00 -> 54.0 mm
- net /VCCA09: track 0.00 -> 44.3 mm
- net /VCCA33: track 0.00 -> 40.7 mm
- net /VACustom: track 0.00 -> 22.5 mm
- net ADGND: vias 0 -> 15
- added copper zone on F.Cu, net /AVIN5
- added copper zone on B.Cu, net ADGND
- added copper zone on B.Cu, net DGND
- added copper zone on F.Cu, net DGND

Commit message: init layout
Parts:
- added R33: 4.7k, Resistor_SMD:R_0805_2012Metric, F.Cu at (229.9, 142.9)
- added R34: 4.7k, Resistor_SMD:R_0805_2012Metric, F.Cu at (229.9, 145.9)
- added REF**: MountingHole_3.5mm, MountingHole:MountingHole_3.5mm, F.Cu at (104.0, 121.0)
- added REF**: MountingHole_3.5mm, MountingHole:MountingHole_3.5mm, F.Cu at (196.0, 30.0)
- added REF**: MountingHole_3.5mm, MountingHole:MountingHole_3.5mm, F.Cu at (104.0, 30.0)
- added REF**: MountingHole_3.5mm, MountingHole:MountingHole_3.5mm, F.Cu at (196.0, 121.0)
- added S8: 2454985-3, 2_DS:24549853, F.Cu at (74.7, 115.9)
- C26, C28, C29, C30, C33, C34, C37, C38, C39, C44, C47, C49, R1, R2, R3, U17: moved to B.Cu
- moved R9 211.1 mm to (49.9, 80.6)
- moved R21 188.5 mm to (65.6, 51.2)
- moved S1 187.4 mm to (82.3, 87.2), turned to 90 degrees
- moved S2 178.2 mm to (77.2, 103.0), turned to 90 degrees
- moved C8 165.3 mm to (108.2, 85.8), turned to 90 degrees
- moved R22 164.0 mm to (84.7, 77.8)
- moved C28 153.0 mm to (108.2, 92.9), turned to 90 degrees
- moved C29 152.7 mm to (108.2, 87.8), turned to -90 degrees
- moved C9 145.5 mm to (134.9, 103.3), turned to -90 degrees
- moved C11 141.5 mm to (137.0, 103.3), turned to 90 degrees
- moved J10 140.8 mm to (157.4, 107.6)
- moved C26 139.7 mm to (122.4, 94.7), turned to -90 degrees
- moved C31 137.9 mm to (108.2, 95.0), turned to -90 degrees
- moved C10 137.7 mm to (142.3, 103.3), turned to -90 degrees
- moved C33 137.5 mm to (108.2, 74.0), turned to 90 degrees
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Connections:
- J10 pad 1: VDCustom -> DGND
- J10 pad 10: DGND -> VCCD12
- J10 pad 11: VCCD33 -> DGND
- J10 pad 12: DGND -> VCCD09
- J10 pad 13: DVIN5 -> DGND
- J10 pad 14: DGND -> VDCustom
- J10 pad 2: DGND -> DVIN5
- J10 pad 3: VCCD09 -> DGND
- J10 pad 4: DGND -> VCCD33
- J10 pad 5: VCCD12 -> DGND
- J10 pad 6: DGND -> VCCD25
- J10 pad 7: VCCD18 -> DGND
- J10 pad 8: DGND -> VCCD18
- J10 pad 9: VCCD25 -> DGND
- J4 pad 1: VDCustom -> DVIN5
- J4 pad 11: VCCD33 -> VCCD09
- J4 pad 13: DVIN5 -> VDCustom
- J4 pad 3: VCCD09 -> VCCD33
- J4 pad 5: VCCD12 -> VCCD25
- J4 pad 9: VCCD25 -> VCCD12
- U12 pad 11: MC2_58 -> MC2_58_PIN
- U12 pad 12: MC2_60 -> MC2_60_PIN
- U12 pad 13: MC2_62 -> MC2_62_PIN
- U12 pad 14: MC2_64 -> MC2_64_PIN
- U12 pad 16: MC2_66 -> MC2_66_PIN
- U12 pad 17: MC2_68 -> MC2_68_PIN
- U12 pad 19: MC2_70 -> MC2_70_PIN
- U12 pad 2: MC2_44 -> MC2_44_PIN
- U12 pad 20: MC2_72 -> MC2_72_PIN
- U12 pad 22: MC2_74 -> MC2_74_PIN
- U12 pad 23: MC2_76 -> MC2_76_PIN
- U12 pad 26: MC2_76_PIN -> MC2_76
- U12 pad 27: MC2_74_PIN -> MC2_74
- U12 pad 29: MC2_72_PIN -> MC2_72
- U12 pad 3: MC2_46 -> MC2_46_PIN
- U12 pad 30: MC2_70_PIN -> MC2_70
- U12 pad 32: MC2_68_PIN -> MC2_68
- U12 pad 33: MC2_66_PIN -> MC2_66
- U12 pad 35: MC2_64_PIN -> MC2_64
- U12 pad 36: MC2_62_PIN -> MC2_62
- U12 pad 37: MC2_60_PIN -> MC2_60
- U12 pad 38: MC2_58_PIN -> MC2_58
- U12 pad 40: MC2_54_PIN -> MC2_54
- U12 pad 41: MC2_52_PIN -> MC2_52
- U12 pad 43: MC2_50_PIN -> MC2_50
- U12 pad 44: MC2_48_PIN -> MC2_48
- U12 pad 46: MC2_46_PIN -> MC2_46
- U12 pad 47: MC2_44_PIN -> MC2_44
- U12 pad 5: MC2_48 -> MC2_48_PIN
- U12 pad 6: MC2_50 -> MC2_50_PIN
- U12 pad 8: MC2_52 -> MC2_52_PIN
- U12 pad 9: MC2_54 -> MC2_54_PIN
- U13 pad 11: MC2_27 -> MC2_25
- U13 pad 12: MC2_29 -> MC2_27
- U13 pad 13: MC2_31 -> MC2_29
- U13 pad 14: MC2_33 -> MC2_31
- U13 pad 16: MC2_37 -> MC2_33
- U13 pad 17: MC2_39 -> MC2_37
- U13 pad 19: MC2_41 -> MC2_39
- U13 pad 2: MC2_15 -> MC2_10
- U13 pad 20: MC2_43 -> MC2_41
- U13 pad 22: MC2_45 -> MC2_43
- U13 pad 23: MC2_10 -> MC2_45
- U13 pad 26: MC2_10_PIN -> MC2_45_PIN
- U13 pad 27: MC2_45_PIN -> MC2_43_PIN
- U13 pad 29: MC2_43_PIN -> MC2_41_PIN
- U13 pad 3: MC2_17 -> MC2_15
- U13 pad 30: MC2_41_PIN -> MC2_39_PIN
- U13 pad 32: MC2_39_PIN -> MC2_37_PIN
- U13 pad 33: MC2_37_PIN -> MC2_33_PIN
- U13 pad 35: MC2_33_PIN -> MC2_31_PIN
- U13 pad 36: MC2_31_PIN -> MC2_29_PIN
- U13 pad 37: MC2_29_PIN -> MC2_27_PIN
- U13 pad 38: MC2_27_PIN -> MC2_25_PIN
- U13 pad 40: MC2_25_PIN -> MC2_23_PIN
- U13 pad 41: MC2_23_PIN -> MC2_21_PIN
- U13 pad 43: MC2_21_PIN -> MC2_19_PIN
- U13 pad 44: MC2_19_PIN -> MC2_17_PIN
- U13 pad 46: MC2_17_PIN -> MC2_15_PIN
- U13 pad 47: MC2_15_PIN -> MC2_10_PIN
- U13 pad 5: MC2_19 -> MC2_17
- U13 pad 6: MC2_21 -> MC2_19
- U13 pad 8: MC2_23 -> MC2_21
- U13 pad 9: MC2_25 -> MC2_23
- U16 pad 11: MC1_64 -> MC1_58
- U16 pad 12: MC1_66 -> MC1_60
- U16 pad 13: MC1_68 -> MC1_62
- U16 pad 14: MC1_70 -> MC1_64
- U16 pad 16: MC1_72 -> MC1_66
- U16 pad 17: MC1_74 -> MC1_68
- U16 pad 19: MC1_76 -> MC1_70
- U16 pad 2: MC1_50 -> MC1_19
- U16 pad 20: MC1_15 -> MC1_72
- U16 pad 22: MC1_17 -> MC1_74
- U16 pad 23: MC1_19 -> MC1_76
- U16 pad 26: MC1_19_PIN -> MC1_76_PIN
- U16 pad 27: MC1_17_PIN -> MC1_74_PIN
- U16 pad 29: MC1_15_PIN -> MC1_72_PIN
- U16 pad 3: MC1_52 -> MC1_17
- U16 pad 30: MC1_76_PIN -> MC1_70_PIN
- U16 pad 32: MC1_74_PIN -> MC1_68_PIN
- U16 pad 33: MC1_72_PIN -> MC1_66_PIN
- U16 pad 35: MC1_70_PIN -> MC1_64_PIN
- U16 pad 36: MC1_68_PIN -> MC1_62_PIN
- U16 pad 37: MC1_66_PIN -> MC1_60_PIN
- U16 pad 38: MC1_64_PIN -> MC1_58_PIN
- U16 pad 40: MC1_62_PIN -> MC1_54_PIN
- U16 pad 41: MC1_60_PIN -> MC1_52_PIN
- U16 pad 43: MC1_58_PIN -> MC1_50_PIN
- U16 pad 44: MC1_54_PIN -> MC1_15_PIN
- U16 pad 46: MC1_52_PIN -> MC1_17_PIN
- U16 pad 47: MC1_50_PIN -> MC1_19_PIN
- U16 pad 5: MC1_54 -> MC1_15
- U16 pad 6: MC1_58 -> MC1_50
- U16 pad 8: MC1_60 -> MC1_52
- U16 pad 9: MC1_62 -> MC1_54
- U17 pad 11: MC1_33 -> MC1_33_PIN
- U17 pad 12: MC1_37 -> MC1_37_PIN
- U17 pad 13: MC1_39 -> MC1_39_PIN
- U17 pad 14: MC1_41 -> MC1_41_PIN
- U17 pad 16: MC1_43 -> MC1_43_PIN
- U17 pad 17: MC1_45 -> MC1_45_PIN
- U17 pad 19: MC1_47 -> MC1_47_PIN
- U17 pad 2: MC1_21 -> MC1_21_PIN
- U17 pad 20: MC1_49 -> MC1_49_PIN
- U17 pad 22: MC1_51 -> MC1_51_PIN
- U17 pad 23: MC1_53 -> MC1_53_PIN
- U17 pad 26: MC1_53_PIN -> MC1_53
- U17 pad 27: MC1_51_PIN -> MC1_51
- U17 pad 29: MC1_49_PIN -> MC1_49
- U17 pad 3: MC1_23 -> MC1_23_PIN
- U17 pad 30: MC1_47_PIN -> MC1_47
- U17 pad 32: MC1_45_PIN -> MC1_45
- U17 pad 33: MC1_43_PIN -> MC1_43
- U17 pad 35: MC1_41_PIN -> MC1_41
- U17 pad 36: MC1_39_PIN -> MC1_39
- U17 pad 37: MC1_37_PIN -> MC1_37
- U17 pad 38: MC1_33_PIN -> MC1_33
- U17 pad 40: MC1_31_PIN -> MC1_31
- U17 pad 41: MC1_29_PIN -> MC1_29
- U17 pad 43: MC1_27_PIN -> MC1_27
- U17 pad 44: MC1_25_PIN -> MC1_25
- U17 pad 46: MC1_23_PIN -> MC1_23
- U17 pad 47: MC1_21_PIN -> MC1_21
- U17 pad 5: MC1_25 -> MC1_25_PIN
- U17 pad 6: MC1_27 -> MC1_27_PIN
- U17 pad 8: MC1_29 -> MC1_29_PIN
- U17 pad 9: MC1_31 -> MC1_31_PIN
Routing:
- net FPGA_GND: track 0.00 -> 133.9 mm
- net VCCD33: track 0.00 -> 96.5 mm, vias 0 -> 1
- net MC1_71_PIN: track 0.00 -> 81.8 mm, vias 0 -> 1
- net VCCD18: track 0.00 -> 80.1 mm, vias 0 -> 1
- net MC1_69_PIN: track 0.00 -> 80.0 mm, vias 0 -> 1
- net MC1_67_PIN: track 0.00 -> 79.2 mm, vias 0 -> 1
- net MC1_65_PIN: track 0.00 -> 77.6 mm, vias 0 -> 1
- net VCCD25: track 0.00 -> 76.2 mm, vias 0 -> 2
- net MC1_63_PIN: track 0.00 -> 76.0 mm, vias 0 -> 1
- net MC1_61_PIN: track 0.00 -> 74.5 mm, vias 0 -> 1
- net FPGA_33VDD: track 0.00 -> 73.6 mm, vias 0 -> 1
- net MC1_59_PIN: track 0.00 -> 72.7 mm, vias 0 -> 1
- net VCCD12: track 0.00 -> 71.9 mm
- net DVIN5: track 0.00 -> 71.7 mm, vias 0 -> 2
- net VCCD09: track 0.00 -> 70.9 mm
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Other:
- board text added: "lower"
- board text added: "swtich sides"

Commit message: progress
Parts:
- removed R27, R28, R31, R32, R33, R34: 4.7k, Resistor_SMD:R_0805_2012Metric
- removed S7, S8: 2454985-3, 2_DS:24549853
- removed U11: SN74LVC16T245DLR, avlsi:DL48
- C22, C23, C24, C25, R16, R21, R22, R25, R26, S2, S3, S4, U15: moved to B.Cu
- C34, C37, C47, C49, U17: moved to F.Cu
- R5, R6: value 10k -> 4.7k
- moved R8 168.8 mm to (108.8, 33.6), turned to 90 degrees
- moved R7 153.5 mm to (123.2, 33.5), turned to 90 degrees
- moved R12 143.9 mm to (108.5, 113.7), turned to -90 degrees
- moved S3 137.7 mm to (115.8, 111.5)
- moved R10 136.1 mm to (126.0, 109.5), turned to 90 degrees
- moved R13 134.5 mm to (112.8, 65.1), turned to 90 degrees
- moved R14 133.3 mm to (112.6, 77.7), turned to -90 degrees
- moved R11 130.0 mm to (123.0, 114.0), turned to -90 degrees
- moved R6 124.9 mm to (108.6, 109.6), turned to 90 degrees
- moved R5 117.7 mm to (123.1, 109.4), turned to 90 degrees
- moved R19 115.9 mm to (172.3, 41.4), turned to 90 degrees
- moved R21 113.1 mm to (178.0, 63.6)
- moved R20 105.7 mm to (186.6, 41.5), turned to 90 degrees
- moved R23 98.6 mm to (172.1, 33.4), turned to 90 degrees
- moved R17 96.5 mm to (112.8, 88.3), turned to 180 degrees
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Connections:
- J5 pad 25: MC2_26_PIN -> MC2_26
- J5 pad 27: MC2_28_PIN -> MC2_28
- J5 pad 29: MC2_30_PIN -> MC2_30
- J5 pad 31: MC2_32_PIN -> MC2_32
- J5 pad 33: MC2_34_PIN -> MC2_34
- J5 pad 37: MC2_38_PIN -> MC2_38
- J5 pad 39: MC2_40_PIN -> MC2_40
- J6 pad 1: MC2_42_PIN -> MC2_42
- J8 pad 18: MC1_57_PIN -> MC1_71
- J8 pad 20: MC1_59_PIN -> MC1_69
- J8 pad 22: MC1_61_PIN -> MC1_67
- J8 pad 24: MC1_63_PIN -> MC1_65
- J8 pad 26: MC1_65_PIN -> MC1_63
- J8 pad 28: MC1_67_PIN -> MC1_61
- J8 pad 30: MC1_69_PIN -> MC1_59
- J8 pad 32: MC1_71_PIN -> MC1_57
- R11 pad 1: /level_shifter1/DIR1 -> /level_shifter3/DIR1
- R12 pad 1: /level_shifter1/DIR2 -> /level_shifter3/DIR2
- R15 pad 1: /level_shifter2/DIR1 -> /level_shifter4/DIR1
- R16 pad 1: /level_shifter2/DIR2 -> /level_shifter4/DIR2
- R19 pad 1: /level_shifter3/DIR1 -> /level_shifter5/DIR1
- R20 pad 1: /level_shifter3/DIR2 -> /level_shifter5/DIR2
- R23 pad 1: /level_shifter4/DIR1 -> /level_shifter6/DIR1
- R24 pad 1: /level_shifter4/DIR2 -> /level_shifter6/DIR2
- R5 pad 1: DGND -> /level_shifter1/DIR1
- R5 pad 2: Net-(U11-*1OE) -> DGND
- R6 pad 1: DGND -> /level_shifter1/DIR2
- R6 pad 2: Net-(U11-*2OE) -> DGND
- R7 pad 1: /level_shifter/DIR1 -> /level_shifter2/DIR1
- R8 pad 1: /level_shifter/DIR2 -> /level_shifter2/DIR2
- S1 pad A1: /level_shifter/DIR2 -> /level_shifter1/DIR2
- S1 pad B1: /level_shifter/DIR1 -> /level_shifter1/DIR1
- S2 pad A1: /level_shifter1/DIR2 -> /level_shifter2/DIR2
- S2 pad B1: /level_shifter1/DIR1 -> /level_shifter2/DIR1
- S3 pad A1: /level_shifter2/DIR2 -> /level_shifter3/DIR2
- S3 pad B1: /level_shifter2/DIR1 -> /level_shifter3/DIR1
- S4 pad A1: /level_shifter3/DIR2 -> /level_shifter4/DIR2
- S4 pad B1: /level_shifter3/DIR1 -> /level_shifter4/DIR1
- S5 pad A1: /level_shifter4/DIR2 -> /level_shifter5/DIR2
- S5 pad B1: /level_shifter4/DIR1 -> /level_shifter5/DIR1
- S6 pad A1: /level_shifter5/DIR2 -> /level_shifter6/DIR2
- S6 pad B1: /level_shifter5/DIR1 -> /level_shifter6/DIR1
- U15 pad 11: MC1_28 -> MC1_28_PIN
- U15 pad 12: MC1_30 -> MC1_30_PIN
- U15 pad 13: MC1_32 -> MC1_32_PIN
- U15 pad 14: MC1_34 -> MC1_34_PIN
- U15 pad 16: MC1_38 -> MC1_38_PIN
- U15 pad 17: MC1_40 -> MC1_40_PIN
- U15 pad 19: MC1_42 -> MC1_42_PIN
- U15 pad 2: MC1_16 -> MC1_16_PIN
- U15 pad 20: MC1_44 -> MC1_44_PIN
- U15 pad 22: MC1_46 -> MC1_46_PIN
- U15 pad 23: MC1_48 -> MC1_48_PIN
- U15 pad 26: MC1_48_PIN -> MC1_48
- U15 pad 27: MC1_46_PIN -> MC1_46
- U15 pad 29: MC1_44_PIN -> MC1_44
- U15 pad 3: MC1_18 -> MC1_18_PIN
- U15 pad 30: MC1_42_PIN -> MC1_42
- U15 pad 32: MC1_40_PIN -> MC1_40
- U15 pad 33: MC1_38_PIN -> MC1_38
- U15 pad 35: MC1_34_PIN -> MC1_34
- U15 pad 36: MC1_32_PIN -> MC1_32
- U15 pad 37: MC1_30_PIN -> MC1_30
- U15 pad 38: MC1_28_PIN -> MC1_28
- U15 pad 40: MC1_26_PIN -> MC1_26
- U15 pad 41: MC1_24_PIN -> MC1_24
- U15 pad 43: MC1_22_PIN -> MC1_22
- U15 pad 44: MC1_20_PIN -> MC1_20
- U15 pad 46: MC1_18_PIN -> MC1_18
- U15 pad 47: MC1_16_PIN -> MC1_16
- U15 pad 5: MC1_20 -> MC1_20_PIN
- U15 pad 6: MC1_22 -> MC1_22_PIN
- U15 pad 8: MC1_24 -> MC1_24_PIN
- U15 pad 9: MC1_26 -> MC1_26_PIN
- U17 pad 11: MC1_33_PIN -> MC1_33
- U17 pad 12: MC1_37_PIN -> MC1_37
- U17 pad 13: MC1_39_PIN -> MC1_39
- U17 pad 14: MC1_41_PIN -> MC1_41
- U17 pad 16: MC1_43_PIN -> MC1_43
- U17 pad 17: MC1_45_PIN -> MC1_45
- U17 pad 19: MC1_47_PIN -> MC1_47
- U17 pad 2: MC1_21_PIN -> MC1_21
- U17 pad 20: MC1_49_PIN -> MC1_49
- U17 pad 22: MC1_51_PIN -> MC1_51
- U17 pad 23: MC1_53_PIN -> MC1_53
- U17 pad 26: MC1_53 -> MC1_53_PIN
- U17 pad 27: MC1_51 -> MC1_51_PIN
- U17 pad 29: MC1_49 -> MC1_49_PIN
- U17 pad 3: MC1_23_PIN -> MC1_23
- U17 pad 30: MC1_47 -> MC1_47_PIN
- U17 pad 32: MC1_45 -> MC1_45_PIN
- U17 pad 33: MC1_43 -> MC1_43_PIN
- U17 pad 35: MC1_41 -> MC1_41_PIN
- U17 pad 36: MC1_39 -> MC1_39_PIN
- U17 pad 37: MC1_37 -> MC1_37_PIN
- U17 pad 38: MC1_33 -> MC1_33_PIN
- U17 pad 40: MC1_31 -> MC1_31_PIN
- U17 pad 41: MC1_29 -> MC1_29_PIN
- U17 pad 43: MC1_27 -> MC1_27_PIN
- U17 pad 44: MC1_25 -> MC1_25_PIN
- U17 pad 46: MC1_23 -> MC1_23_PIN
- U17 pad 47: MC1_21 -> MC1_21_PIN
- U17 pad 5: MC1_25_PIN -> MC1_25
- U17 pad 6: MC1_27_PIN -> MC1_27
- U17 pad 8: MC1_29_PIN -> MC1_29
- U17 pad 9: MC1_31_PIN -> MC1_31
Routing:
- net FPGA_GND: track 133.9 -> 428.3 mm, vias 0 -> 6
- net FPGA_33VDD: track 73.6 -> 243.9 mm, vias 1 -> 6
- net MC1_71_PIN: track 81.8 -> 0.00 mm, vias 1 -> 0
- net MC1_69_PIN: track 80.0 -> 0.00 mm, vias 1 -> 0
- net MC1_67_PIN: track 79.2 -> 0.00 mm, vias 1 -> 0
- net MC1_65_PIN: track 77.6 -> 0.00 mm, vias 1 -> 0
- net MC1_63_PIN: track 76.0 -> 0.00 mm, vias 1 -> 0
- net MC1_61_PIN: track 74.5 -> 0.00 mm, vias 1 -> 0
- net MC1_59_PIN: track 72.7 -> 0.00 mm, vias 1 -> 0
- net MC1_57_PIN: track 70.7 -> 0.00 mm, vias 1 -> 0
- net /level_shifter5/DIR2: track 0.00 -> 64.1 mm, vias 0 -> 4
- net /level_shifter6/DIR2: track 0.00 -> 60.2 mm, vias 0 -> 2
- net /level_shifter4/DIR2: track 0.00 -> 58.9 mm, vias 0 -> 2
- net /level_shifter2/DIR2: track 0.00 -> 54.5 mm, vias 0 -> 2
- net /level_shifter5/DIR1: track 0.00 -> 48.9 mm, vias 0 -> 2
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- added copper zone on In2.Cu, net /VCCA33
- added copper zone on F.Cu, net V_Level_Shift
- added copper zone on In1.Cu, net V_Level_Shift
- removed copper zone on F.Cu, net DGND
Other:
- board text removed: "lower"
- board text removed: "swtich sides"
