File: avlsi_test_boards/power_board/power_board.kicad_sch (KiCad schematic)
At the start: 9 parts, among them J1 PJ-102AH, J10 Conn_02x07_Odd_Even, J2 PJ-102AH, J3 Conn_02x07_Odd_Even, J4 Conn_02x07_Odd_Even, J9 Conn_02x07_Odd_Even

Commit message: progress
Parts:
- removed R33, R34: 4.7k, Resistor_SMD:R_0805_2012Metric, symbol Device:R
- removed S8: 2454985-3, 2_DS:24549853, symbol 2_DIP:2454985-3
Other:
- removed sheet level_shifter
