File: avlsi_test_boards/power_board/digital_power_converters.kicad_sch (KiCad schematic)
At the start: 21 parts, among them U1 TLV1117LV18DCYR, U11 TLV75709PDBV, U2 TLV1117LV25DCYR, U3 TLV1117LV33DCYR, U4 DS04-254-2-04BK-SMT, U5 74HC4051D_653

Commit message: Update schematic
Connections:
- net DGND: now also U5.6 (~E)
- net DVIN5: no longer U5.6 (~E)
Changed lines of the file:
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@@
-	)
-	(junction
-		(at 186.69 114.3)
-		(diameter 0)
-		(color 0 0 0 0)
 	)
 	(junction
@@
 	)
 	(junction
+		(at 175.26 134.62)
+		(diameter 0)
+		(color 0 0 0 0)
+	)
+	(junction
 		(at 59.69 74.93)
 		(diameter 0)
@@
 	(wire
 		(pts
-			(xy 186.69 119.38) (xy 190.5 119.38)
-		)
-		(stroke
-			(width 0)
-			(type default)
-		)
-	)
-	(wire
-		(pts
-			(xy 167.64 114.3) (xy 186.69 114.3)
+			(xy 167.64 114.3) (xy 190.5 114.3)
 		)
 		(stroke
@@
 	(wire
 		(pts
-			(xy 167.64 134.62) (xy 184.15 134.62)
+			(xy 167.64 134.62) (xy 175.26 134.62)
 		)
 		(stroke
@@
 	(wire
 		(pts
+			(xy 175.26 119.38) (xy 190.5 119.38)
+		)
+		(stroke
+			(width 0)
+			(type default)
+		)
+	)
+	(wire
+		(pts
 			(xy 257.81 78.74) (xy 259.08 78.74)
 		)
@@
 	(wire
 		(pts
-			(xy 186.69 114.3) (xy 186.69 119.38)
-		)
-		(stroke
-			(width 0)
-			(type default)
-		)
-	)
-	(wire
-		(pts
 			(xy 59.69 161.29) (xy 59.69 165.1)
 		)
@@
 	(wire
 		(pts
-			(xy 186.69 114.3) (xy 190.5 114.3)
-		)
-		(stroke
-			(width 0)
-			(type default)
-		)
-	)
-	(wire
-		(pts
 			(xy 226.06 121.92) (xy 248.92 121.92)
 		)
@@
 	(wire
 		(pts
+			(xy 175.26 119.38) (xy 175.26 134.62)
+		)
+		(stroke
+			(width 0)
+			(type default)
+		)
+	)
+	(wire
+		(pts
 			(xy 59.69 124.46) (xy 59.69 128.27)
 		)
@@
 		)
 		(stroke
+			(width 0)
+			(type default)
+		)
+	)
+	(wire
+		(pts
+			(xy 175.26 134.62) (xy 184.15 134.62)
+		)
+		(stroke
